Commit message: remove box

File: iiwa_tool/iiwa_tool_description/urdf/iiwa7_simple_tool.urdf.xacro (robot description, xacro)
@@ -9,24 +9,5 @@
     <xacro:arg name="hardware_interface" default="PositionJointInterface"/>
     <xacro:arg name="robot_name" default="iiwa"/>
-    <!--  Define the origin of your 3D space
-    Here we define a box lying at 0,0,0 with some dimensions, in reality our robot is place on top of a metal cart with those dimensions.
-    This will include the cart in the scene and avoid the robot to hit it when using MoveIt!
-    If you don't want to have that you can define a basic world link (see commented lines)
-    -->
-    <!--     <link name="world"/> -->
-    <link name="world">
-        <visual>
-            <origin xyz="0 0 0.42" rpy="0 0 0"/>
-            <geometry>
-                <box size="0.68 0.605 0.84"/>
-            </geometry>
-        </visual>
-        <collision>
-            <origin xyz="0 0 0.42" rpy="0 0 0"/>
-            <geometry>
-                <box size="0.68 0.605 0.84"/>
-            </geometry>
-        </collision>
-    </link>
+    <link name="world"/>
     <gazebo reference="world">
         <static>true</static>
@@ -34,5 +15,5 @@
     <!-- Here we insert an iiwa7 robot in the scene, it's origin is just on top of the box previously defined. You can use 0,0,0 if you don't have that. -->
     <xacro:iiwa7 hardware_interface="$(arg hardware_interface)" robot_name="$(arg robot_name)" parent="world">
-        <origin xyz="0 0 0.84" rpy="0 0 0"/>
+        <origin xyz="0 0 0" rpy="0 0 0"/>
     </xacro:iiwa7>
     <!-- Tool properties -->
