Commit message: add RCM to tf and iiwa_link0 to the planning group

File: iiwa_tool/iiwa_needle_description/urdf/iiwa7_needle.urdf.xacro (robot description, xacro)
@@ -60,3 +60,9 @@
     <!--  The TCP frame is here defined -->
     <link name="tool_link_ee"/>
+    <link name="RCM"/>
+    <joint name="RCM_JOINT" type="fixed">
+        <parent link="world"/>
+        <child link="RCM"/>
+        <origin xyz="0 -0.5 0.3" rpy="0 0 0"/>
+    </joint>
 </robot>

File: iiwa_tool/iiwa_needle_moveit/config/gazebo_iiwa7_tool.urdf (robot description, URDF)
Before this commit: robot iiwa7_tool, 12 links, 11 joints
Links:
- added link RCM
Joints:
- added joint RCM_JOINT: type fixed, parent world, child RCM, origin xyz=0 -0.5 0.3 rpy=0 0 0

Commit message: successful tool insertion

File: iiwa_tool/iiwa_needle_description/urdf/iiwa7_needle.urdf.xacro (robot description, xacro)
@@ -60,9 +60,21 @@
     <!--  The TCP frame is here defined -->
     <link name="tool_link_ee"/>
+    <link name="abdomen_base"/>
+    <joint name="abdomen_base_joint" type="fixed">
+        <parent link="world"/>
+        <child link="abdomen_base"/>
+        <origin xyz="0 -0.5 0.0" rpy="0 0 0"/>
+    </joint>
     <link name="RCM"/>
     <joint name="RCM_JOINT" type="fixed">
-        <parent link="world"/>
+        <parent link="abdomen_base"/>
         <child link="RCM"/>
-        <origin xyz="0 -0.5 0.3" rpy="0 0 0"/>
+        <origin xyz="0 0.0 0.3" rpy="0 0 0"/>
+    </joint>
+    <link name="Insertion_Pose"/>
+    <joint name="INSERTION_JOINT" type="fixed">
+        <parent link="RCM"/>
+        <child link="Insertion_Pose"/>
+        <origin xyz="0 0 0" rpy="0 ${pi} 0"/>
     </joint>
 </robot>

File: iiwa_tool/iiwa_needle_moveit/config/gazebo_iiwa7_tool.urdf (robot description, URDF)
Before this commit: robot iiwa7_tool, 13 links, 12 joints
Links:
- added link Insertion_Pose
Joints:
- added joint INSERTION_JOINT: type fixed, parent RCM, child Insertion_Pose, origin xyz=0 0 0 rpy=0 3.141592653589793 0

Commit message: increase needle length

File: iiwa_tool/iiwa_needle_description/urdf/iiwa7_needle.urdf.xacro (robot description, xacro)
@@ -37,16 +37,15 @@
         <visual>
             <material name="Grey"/>
-            <origin xyz="0 0 -0.005" rpy="0 ${-pi/2} 0"/>
+            <origin xyz="0 0 0.0" rpy="0 ${-pi/2} 0"/>
             <geometry>
                 <mesh filename="package://iiwa_needle_description/meshes/visual/needle.obj" scale="0.001 0.001 0.001"/>
-                <cylinder length="0.25" radius="0.008"/>
             </geometry>
             <material name="StainlessSteel"/>
         </visual>
         <collision>
-            <origin xyz="0 0 ${0.070 / 2}" rpy="0 0 0"/>
+            <origin xyz="0 0 ${0.150 / 2}" rpy="0 0 0"/>
             <geometry>
                 <!--<mesh filename="package://iiwa_needle_description/meshes/collision/needle.obj" scale="0.001 0.001 0.001"/>-->
-                <cylinder length="0.070" radius="0.004"/>
+                <cylinder length="0.150" radius="0.004"/>
             </geometry>
         </collision>
@@ -56,5 +55,5 @@
         <parent link="tool_link"/>
         <child link="tool_link_ee"/>
-        <origin xyz="0.00 0.00 0.075" rpy="0 0 0"/>
+        <origin xyz="0.00 0.00 0.150" rpy="0 0 0"/>
     </joint>
     <!--  The TCP frame is here defined -->

Commit message: change to a longer needle and refactor code

File: iiwa_tool/iiwa_needle_description/urdf/iiwa7_needle.urdf.xacro (robot description, xacro)
@@ -34,4 +34,5 @@
     <!-- Here we define the geometry of the tool. We designed the tool ourselves, so we have a mesh file that represents it.
     Else, one can define it using a geometric representation that approximate it, like a cylinder (see commented lines) -->
+    <xacro:property name="needle_len" value="0.350"/>
     <link name="tool_link">
         <visual>
@@ -44,8 +45,8 @@
         </visual>
         <collision>
-            <origin xyz="0 0 ${0.150 / 2}" rpy="0 0 0"/>
+            <origin xyz="0 0 ${needle_len / 2}" rpy="0 0 0"/>
             <geometry>
                 <!--<mesh filename="package://iiwa_needle_description/meshes/collision/needle.obj" scale="0.001 0.001 0.001"/>-->
-                <cylinder length="0.150" radius="0.004"/>
+                <cylinder length="${needle_len}" radius="0.004"/>
             </geometry>
         </collision>
@@ -55,5 +56,5 @@
         <parent link="tool_link"/>
         <child link="tool_link_ee"/>
-        <origin xyz="0.00 0.00 0.150" rpy="0 0 0"/>
+        <origin xyz="0.00 0.00 ${needle_len}" rpy="0 0 0"/>
     </joint>
     <!--  The TCP frame is here defined -->

File: iiwa_tool/iiwa_needle_moveit/config/gazebo_iiwa7_tool.urdf (robot description, URDF)
Before this commit: robot iiwa7_tool, 14 links, 13 joints
Links:
- added link abdomen_base
- link tool_link: geometry collision cylinder length=0.35 radius=0.004; visual mesh filename=package://iiwa_needle_description/meshes/visual/needle.obj scale=0.001 0.001 0.001
Joints:
- added joint abdomen_base_joint: type fixed, parent world, child abdomen_base, origin xyz=0 -0.5 0.0 rpy=0 0 0
- joint RCM_JOINT: origin xyz=0 -0.5 0.3 rpy=0 0 0 -> xyz=0 0.0 0.3 rpy=0 0 0; parent world -> abdomen_base
- joint tool_tip_joint: origin xyz=0.00 0.00 0.075 rpy=0 0 0 -> xyz=0.00 0.00 0.35 rpy=0 0 0

Commit message: update needle radius

File: iiwa_tool/iiwa_needle_description/urdf/iiwa7_needle.urdf.xacro (robot description, xacro)
@@ -48,5 +48,5 @@
             <geometry>
                 <!--<mesh filename="package://iiwa_needle_description/meshes/collision/needle.obj" scale="0.001 0.001 0.001"/>-->
-                <cylinder length="${needle_len}" radius="0.004"/>
+                <cylinder length="${needle_len}" radius="0.002"/>
             </geometry>
         </collision>

Commit message: move rcm to (x=0.5)

File: iiwa_tool/iiwa_needle_description/urdf/iiwa7_needle.urdf.xacro (robot description, xacro)
@@ -64,5 +64,5 @@
         <parent link="world"/>
         <child link="abdomen_base"/>
-        <origin xyz="0 -0.5 0.0" rpy="0 0 0"/>
+        <origin xyz="0.5 0.0 0.0" rpy="0 0 0"/>
     </joint>
     <link name="RCM"/>
